File: STM32 keyboard Module_v1.kicad_pcb (KiCad board)
At the start: 4 copper layers, 49.2 x 35.7 mm, 48 parts, among them J1 TC2030, J10 PINHD_1x1, J11 PINHD_1x1, J3 PINHD_1x19, J4 PINHD_1x19, J5 Castellated_PINHD_1x20, J6 Castellated_PINHD_1x20, J7 PINHD_1x1, J8 PINHD_1x1, J9 PINHD_1x1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

Commit message: Second commit
Parts:
- renumbered locked to J2
