File: STM32 keyboard Module.kicad_pcb (KiCad board)
At the start: 4 copper layers, 49.1 x 28.2 mm, 48 parts, among them J1 TC2030, J10 PINHD_1x1, J11 PINHD_1x1, J3 PINHD_1x19, J4 PINHD_1x19, J5 Castellated_PINHD_1x20, J6 Castellated_PINHD_1x20, J7 PINHD_1x1, J8 PINHD_1x1, J9 PINHD_1x1, SW1 PTS815 SJM 250 SMTR LFS, SW2 PTS815 SJM 250 SMTR LFS, U1 LD39050PU33R, U2 STM32U575VGT6, X1 48Mhz, X2 32khz

Commit message: Second commit
Parts:
- J1: moved to B.Cu
- moved J10 25.7 mm to (55.0, 38.4), turned to 180 degrees
- moved J11 25.4 mm to (56.5, 38.4), turned to 180 degrees
- moved X2 4.95 mm to (85.8, 54.0)
- moved FID1 3.04 mm to (59.6, 39.0)
- moved C23 1.71 mm to (64.6, 40.8), turned to 180 degrees
- moved C8 1.36 mm to (63.0, 55.6), turned to 180 degrees
- moved FID3 0.81 mm to (91.9, 39.1)
- moved C18 0.70 mm to (56.9, 42.6), turned to 0 degrees
- moved X1 0.70 mm to (86.5, 50.0)
- moved C4 0.69 mm to (82.8, 54.3), turned to -90 degrees
- moved C10 0.65 mm to (63.0, 56.5), turned to 180 degrees
- moved C7 0.53 mm to (63.8, 42.7)
- moved FID2 0.38 mm to (91.8, 63.2)
- moved C5 0.16 mm to (83.3, 51.5)
- turned J1 to 180 degrees
- renumbered locked to J2
Routing:
- net +5V: track 32.6 -> 15.8 mm, vias 6 -> 5
- net /LSE_OUT: track 10.6 -> 5.55 mm
- net /LSE_IN: track 10.6 -> 5.92 mm
- net I2C_2_SCL: track 19.1 -> 22.3 mm
- net Net-(U2-VCAP): track 7.12 -> 4.44 mm
- net /PIN_38: track 18.6 -> 21.0 mm
- net /HSE_IN: track 7.10 -> 4.98 mm
- net +3.3V: track 31.7 -> 33.8 mm, vias 19 -> 18
- net /SWD_SWCLK: track 7.61 -> 8.89 mm, vias 0 -> 1
- net GND: track 40.6 -> 41.8 mm, vias 49 -> 46
- net NRST: track 46.9 -> 47.9 mm
- net USART 3 TX: track 21.4 -> 20.3 mm
- net /PIN_52: track 17.0 -> 17.9 mm
- net Net-(D2-L2): track 14.0 -> 13.2 mm
- net USART 1 CK: track 10.9 -> 11.7 mm
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
Commit message: Board v2
Parts:
- removed the C11 at (90.3, 47.2)
- removed the C9 at (83.3, 59.5)
- removed the R1 at (86.7, 60.0)
- added C15: 4.7uF, Capacitor_SMD:C_0603_1608Metric, F.Cu at (64.8, 40.9)
- added C17: 10uF, Capacitor_SMD:C_0603_1608Metric, F.Cu at (83.5, 57.7)
- added J12: PINHD_1x4, Wolffyx:Castellated_PinHeader_1x4_P1.27mm_1_1_1, F.Cu at (56.7, 64.5)
- added J13: PINHD_1x1, Wolffyx:Castellated_PinHeader_1x1_P1.27mm_1_1, F.Cu at (61.8, 64.5)
- added R3: 220R, Resistor_SMD:R_0402_1005Metric, F.Cu at (86.3, 59.4)
- C1: value 10nF -> 100nF; footprint Capacitor_SMD:C_0603_1608Metric -> Capacitor_SMD:C_0402_1005Metric
- C12, C3: value 10uF -> 100nF; footprint Capacitor_SMD:C_0603_1608Metric -> Capacitor_SMD:C_0402_1005Metric
- C13: value 100nF -> 10nF; footprint Capacitor_SMD:C_0402_1005Metric -> Capacitor_SMD:C_0603_1608Metric
- C14: value 100nF -> 1uF; footprint Capacitor_SMD:C_0402_1005Metric -> Capacitor_SMD:C_0603_1608Metric
- C19: value 16pF -> 100nF
- C2: value 1uF -> 100nF; footprint Capacitor_SMD:C_0603_1608Metric -> Capacitor_SMD:C_0402_1005Metric
- C21: value 19pF -> 16pF
- C23: value 4.7uF -> 19pF; footprint Capacitor_SMD:C_0603_1608Metric -> Capacitor_SMD:C_0402_1005Metric
- C8: value 100nF -> 10uF; footprint Capacitor_SMD:C_0402_1005Metric -> Capacitor_SMD:C_0603_1608Metric
- SW1, SW2: footprint WolffyxLibrary:SW4_PTS815 SJM 250 SMTR LFS_CNK -> Wolffyx:SW4_PTS815 SJM 250 SMTR LFS_CNK
- U2: footprint Package_QFP:LQFP-100_14x14mm_P0.5mm -> STM32U575VGT6:LQFP-100_STM
- moved FID2 37.5 mm to (54.7, 57.7)
- moved C18 33.0 mm to (85.3, 59.4), turned to 90 degrees
- moved C16 29.8 mm to (82.9, 58.9), turned to 0 degrees
- moved C12 28.4 mm to (57.7, 42.0)
- moved C23 25.9 mm to (87.5, 53.0), turned to 0 degrees
- moved C2 25.4 mm to (63.0, 55.8), turned to -90 degrees
- moved C8 22.6 mm to (83.5, 45.9), turned to 0 degrees
- moved C6 22.3 mm to (63.9, 55.8)
- moved C3 17.9 mm to (78.5, 41.1)
- moved C14 17.3 mm to (84.2, 42.8)
- moved SW2 15.2 mm to (87.0, 43.6), turned to -90 degrees
- moved C10 14.9 mm to (59.5, 42.0)
- moved SW1 14.4 mm to (88.8, 58.0), turned to 90 degrees
- moved FID1 7.04 mm to (54.5, 43.9)
- moved C21 5.72 mm to (86.8, 50.0)
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- renumbered C17 to C11, C15 to C9, D2 to D1, D1 to D2, J8 to J10, J7 to J11, J4 to J2, J6 to J3, J10 to J5, J5 to J6, J2 to J7, J3 to J8, R3 to R1
Connections:
- net /PIN_42 renamed /PD11
- net /PIN_74 renamed /PE0
- net /PIN_75 renamed /PE1
- C12 pad 1: +3.3V -> +5V
- C14 pad 1: /BOOT0 -> +3.3V
- C18 pad 1: +5V -> /BOOT0
- C19 pad 1: /HSE_IN -> NRST
- C20 pad 1: /HSE_OUT -> /HSE_IN
- C21 pad 1: /LSE_IN -> /HSE_OUT
- C22 pad 1: /LSE_OUT -> /LSE_IN
- C23 pad 1: Net-(U2-VCAP) -> /LSE_OUT
- D1 pad 1: Net-(D2-L1) -> /USB_D-
- D1 pad 3: Net-(D2-L2) -> /USB_D+
- J6 pad 13: /PIN_45 -> /USB_D-
- J6 pad 14: /PIN_46 -> /USB_D+
- J6 pad 15: /PIN_47 -> /PD14
- J6 pad 16: /PIN_48 -> /PD15
- J6 pad 17: /PIN_49 -> /PIN_47
- J6 pad 18: /PIN_50 -> /PIN_48
- J6 pad 19: /PIN_51 -> /PIN_49
- J6 pad 20: Net-(D2-L1) -> /PIN_50
- J7 pad 1: Net-(D2-L2) -> /PIN_51
- SW1 pad 1: NRST -> Net-(R3-Pad2)
- SW1 pad 2: NRST -> Net-(R3-Pad2)
- SW1 pad 3: GND -> +3.3V
- SW1 pad 4: GND -> +3.3V
- SW2 pad 1: Net-(R1-Pad2) -> NRST
- SW2 pad 2: Net-(R1-Pad2) -> NRST
- SW2 pad 3: +3.3V -> GND
- SW2 pad 4: +3.3V -> GND
- U2 pad 48: Net-(U2-VCAP) -> Net-(U2C-VCAP)
- U2 pad 61: /PIN_45 -> /PD14
- U2 pad 62: /PIN_46 -> /PD15
Routing:
- net /SWD_SWDIO: track 9.00 -> 28.0 mm
- net /PD15: track 0.00 -> 18.4 mm, vias 0 -> 1
- net /PD14: track 0.00 -> 18.2 mm, vias 0 -> 1
- net /PIN_46: track 16.7 -> 0.00 mm
- net /PIN_45: track 16.4 -> 0.00 mm
- net Net-(D2-L1): track 13.6 -> 0.00 mm
- net Net-(D2-L2): track 13.2 -> 0.00 mm
- net GND: track 41.8 -> 29.5 mm, vias 46 -> 41
- net /SWD_SWCLK: track 8.89 -> 20.1 mm
- net /SWD_SWO: track 16.3 -> 26.9 mm
- net /USB_D+: track 6.15 -> 15.3 mm
- net /USB_D-: track 6.05 -> 15.0 mm
- net NRST: track 47.9 -> 54.9 mm
- net Net-(R3-Pad2): track 0.00 -> 6.86 mm
- net Net-(R1-Pad2): track 5.89 -> 0.00 mm, vias 2 -> 0
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Other:
- board size 49.1 x 28.2 mm -> 44.4 x 28.3 mm
- board text added: "3.3v"
- board text added: "5V"
- board text added: "NRST"
- board text added: "SWCLK"
- board text added: "SWDIO"
- board text added: "SWO"
- board text added: "USB+"
- board text added: "USB-"
