File: STM32 keyboard Module.kicad_sch (KiCad schematic)
At the start: 48 parts, among them J1 TC2030, J10 PINHD_1x1, J11 PINHD_1x1, J2 PINHD_1x1, J3 PINHD_1x19, J4 PINHD_1x19, J5 Castellated_PINHD_1x20, J6 Castellated_PINHD_1x20, J7 PINHD_1x1, J8 PINHD_1x1, J9 PINHD_1x1, SW1 PTS815 SJM 250 SMTR LFS, SW2 PTS815 SJM 250 SMTR LFS, U1 LD39050PU33R, U2 STM32U575VGT6, X1 48Mhz, X2 32khz

Commit message: Board v2
Parts:
- removed C?: 4.7uF, Capacitor_SMD:C_0603_1608Metric, symbol Device:C
- removed C? (x10): 100nF, Capacitor_SMD:C_0402_1005Metric, symbol Device:C
- removed C? (x2): 10uF, Capacitor_SMD:C_0603_1608Metric, symbol Device:C
- removed C?: 10nF, Capacitor_SMD:C_0603_1608Metric, symbol Device:C
- removed C?: 1uF, Capacitor_SMD:C_0603_1608Metric, symbol Device:C
- removed R1: 220R, Resistor_SMD:R_0402_1005Metric, symbol Device:R
- removed U2: STM32U575VGT6, Package_QFP:LQFP-100_14x14mm_P0.5mm, symbol MCU_ST_STM32U5:STM32U575VGTx
- added C1, C16, C18, C2, C3, C4, C5, C6, C7: 100nF, Capacitor_SMD:C_0402_1005Metric, symbol Device:C
- added C13: 10nF, Capacitor_SMD:C_0603_1608Metric, symbol Device:C
- added C14, C17: 1uF, Capacitor_SMD:C_0603_1608Metric, symbol Device:C
- added C15: 4.7uF, Capacitor_SMD:C_0603_1608Metric, symbol Device:C
- added C23: 19pF, Capacitor_SMD:C_0402_1005Metric, symbol Device:C
- added C8: 10uF, Capacitor_SMD:C_0603_1608Metric, symbol Device:C
- added J12: PINHD_1x4, Wolffyx:Castellated_PinHeader_1x4_P1.27mm_1_1_1, symbol Wolffyx:Castellated_PinHeader_1x4
- added J13: PINHD_1x1, Wolffyx:Castellated_PinHeader_1x1_P1.27mm_1_1, symbol Wolffyx:Castellated_PinHeader_1x1
- added R3: 220R, Resistor_SMD:R_0402_1005Metric, symbol Device:R
- added U2: STM32U575VGT6, LQFP-100_STM, symbol STM32U575VGT6_2024-07-23:STM32U575VGT6
- C19: value 16pF -> 100nF; Distribuitor Link https://ro.mouser.com/ProductDetail/Murata-Electronics/GCM1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 -> https://ro.mouser.com/ProductDetail/KYOCERA-AVX/0402ZD104KA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; Manufacturer Murata -> KYOCERA AVX; Manufacturer Part No GCM1555C1H160FA16D -> 0402ZD104KAT2A
- C21: value 19pF -> 16pF; Distribuitor Link https://ro.mouser.com/ProductDetail/Murata-Electronics/GJM1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 -> https://ro.mouser.com/ProductDetail/Murata-Electronics/GCM1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; Manufacturer Part No GJM1555C1H190FB01D -> GCM1555C1H160FA16D
- SW1, SW2: footprint WolffyxLibrary:SW4_PTS815 SJM 250 SMTR LFS_CNK -> Wolffyx:SW4_PTS815 SJM 250 SMTR LFS_CNK
- renumbered D2 to D1, D1 to D2, J8 to J10, J7 to J11, J4 to J2, J6 to J3, J11 to J4, J10 to J5, J5 to J6, J2 to J7, J3 to J8, R3 to R1
Connections:
- net +3.3V: now also SW1.3, SW1.4, C1.1, C13.1, C14.1, C16.1, C17.1, C2.1, C3.1, C4.1, C5.1, C6.1, C7.1, C8.1, J13.1, U2.100 (VDD), U2.11 (VDD), U2.21 (VREF+), U2.22 (VDDA), U2.28 (VDD), U2.50 (VDD), U2.6 (VBAT), U2.73 (VDDUSB), U2.75 (VDD); no longer SW2.3, SW2.4
- net BOOT0: now also C18.1, R3.1, U2.94 (PH3-BOOT0)
- net GND: now also SW2.3, SW2.4, C1.2, C13.2, C14.2, C15.2, C16.2, C17.2, C18.2, C2.2, C23.2, C3.2, C4.2, C5.2, C6.2, C7.2, C8.2, U2.10 (VSS), U2.19 (VSSA), U2.20 (VREF-), U2.27 (VSS), U2.49 (VSS), U2.74 (VSS), U2.99 (VSS); no longer SW1.3, SW1.4
- net HSE_IN: now also C20.1, U2.12 (PH0-OSC_IN); no longer C19.1
- net HSE_OUT: now also C21.1, U2.13 (PH1-OSC_OUT); no longer C20.1
- net I2C_1_SCL: now also U2.95 (PB8)
- net I2C_1_SDA: now also U2.96 (PB9)
- net I2C_2_SCL: now also U2.52 (PB13)
- net I2C_2_SDA: now also U2.53 (PB14)
- net I2C_3_SCL: now also U2.15 (PC0)
- net I2C_3_SDA: now also U2.16 (PC1)
- net I2C_4_SCL: now also U2.59 (PD12)
- net I2C_4_SDA: now also U2.60 (PD13)
- net LSE_IN: now also C22.1, U2.8 (PC14-OSC32_IN); no longer C21.1
- net LSE_OUT: now also C23.1, U2.9 (PC15-OSC32_OUT); no longer C22.1
- net NRST: now also C19.1, SW2.1, SW2.2, J12.4, U2.14 (NRST); no longer SW1.1, SW1.2
- net PD11: now also U2.58 (PD11)
- net PD14: now also J6.15, U2.61 (PD14); no longer J6.13
- net PD15: now also J6.16, U2.62 (PD15); no longer J6.14
- net PE0: now also U2.97 (PE0)
- net PE1: now also U2.98 (PE1)
- net PIN_10: now also U2.17 (PC2)
- net PIN_11: now also U2.18 (PC3)
- net PIN_12: now also U2.23 (PA0)
- net PIN_13: now also U2.24 (PA1)
- net PIN_14: now also U2.25 (PA2)
- net PIN_15: now also U2.26 (PA3)
- net PIN_16: now also U2.29 (PA4)
- net PIN_17: now also U2.30 (PA5)
- net PIN_18: now also U2.31 (PA6)
- net PIN_19: now also U2.32 (PA7)
- net PIN_2: now also U2.1 (PE2)
- net PIN_20: now also U2.33 (PC4)
- net PIN_21: now also U2.34 (PC5)
- net PIN_22: now also U2.35 (PB0)
- net PIN_23: now also U2.36 (PB1)
- net PIN_24: now also U2.37 (PB2)
- net PIN_25: now also U2.38 (PE7)
- net PIN_26: now also U2.39 (PE8)
- net PIN_27: now also U2.40 (PE9)
- net PIN_28: now also U2.41 (PE10)
- net PIN_29: now also U2.42 (PE11)
- net PIN_3: now also U2.2 (PE3)
- net PIN_30: now also U2.43 (PE12)
- net PIN_34: now also U2.47 (PB10)
- net PIN_35: now also U2.51 (PB12)
- net PIN_38: now also U2.54 (PB15)
- net PIN_4: now also U2.3 (PE4)
- net PIN_47: now also J6.17, U2.63 (PC6); no longer J6.15
- net PIN_48: now also J6.18, U2.64 (PC7); no longer J6.16
- net PIN_49: now also J6.19, U2.65 (PC8); no longer J6.17
- net PIN_5: now also U2.4 (PE5)
- net PIN_50: now also J6.20, U2.66 (PC9); no longer J6.18
- net PIN_51: now also J7.1, U2.67 (PA8); no longer J6.19
- net PIN_52: now also U2.68 (PA9)
- net PIN_53: now also U2.69 (PA10)
- net PIN_56: now also U2.77 (PA15)
- net PIN_57: now also U2.78 (PC10)
- net PIN_58: now also U2.79 (PC11)
- net PIN_59: now also U2.80 (PC12)
- net PIN_6: now also U2.5 (PE6)
- net PIN_60: now also U2.81 (PD0)
- net PIN_61: now also U2.82 (PD1)
- net PIN_62: now also U2.83 (PD2)
- net PIN_63: now also U2.84 (PD3)
- net PIN_64: now also U2.85 (PD4)
- net PIN_68: now also U2.90 (PB4)
- net PIN_7: now also U2.7 (PC13)
- net SPI1_MISO: now also U2.45 (PE14)
- net SPI1_MOSI: now also U2.46 (PE15)
- net SPI1_SCK: now also U2.44 (PE13)
- net SWD_SWCLK: now also J12.2, U2.76 (PA14)
- net SWD_SWDIO: now also J12.3, U2.72 (PA13)
- net SWD_SWO: now also J12.1, U2.89 (PB3)
- net USART 1 CK: now also U2.93 (PB7)
- net USART 1 RX: now also U2.92 (PB6)
- net USART 1 TX: now also U2.91 (PB5)
- net USART 2 CK: now also U2.88 (PD7)
- net USART 2 RX: now also U2.87 (PD6)
- net USART 2 TX: now also U2.86 (PD5)
- net USART 3 CK: now also U2.57 (PD10)
- net USART 3 RX: now also U2.56 (PD9)
- net USART 3 TX: now also U2.55 (PD8)
- net USB_D+: now also D1.3 (L2), J6.14, U2.71 (PA12)
- net USB_D-: now also D1.1 (L1), J6.13, U2.70 (PA11)
- new net: R3.2, SW1.1, SW1.2
- new net: C15.1, U2.48 (VCAP)
Other:
- note added: "Power"
- note removed: "PIN_54_D+"
- note removed: "PIN_54_D-"
- moved on the sheet: C?, D1, D2, FID1, FID2, FID3, J10, J11, J2, J3, J4, J5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
